Commit message: Problem with left and right xacro wheels from launch. Done through adding other files.

File: urdf/robot.xacro (robot description, xacro)
@@ -1,6 +1,8 @@
-<robot name = "robot">
+<?xml version="1.0"?>
+<robot xmlns:xacro="http://www.ros.org/wiki/xacro" name="robot">
 <!--  position wrt parent == origin; orientation == rpy  -->
 <!--  units are in meters  -->
 <!--  if you do not put in an origin, it defaults to the COM  -->
+ <!--LINKS-->
         <link name = "base">
                 <visual>
@@ -73,7 +75,9 @@
 	        </collision>
         </link>
-        <link name = "wheel_left">
+ <!--WHEELS-->
+<xacro:macro name="xacro_name" params="suffix reflect">
+        <link name = "wheel_${suffix}">
 	        <visual>
-	                <!--<origin xyz="0 0 0" rpy="-0.0012068 0.114646 -0.0015308"/>-->
+	                <origin xyz="-0.10 ${reflect * 0.4} 0" />
 	                <geometry>
 	                        <cylinder radius="0.2" length="0.05"/>
@@ -81,5 +85,5 @@
  	                </visual>
 	        <collision>
-	                <!--<origin xyz="0 0 0" rpy="-0.0012068 0.114646 -0.0015308"/> -->
+	                <origin xyz="-0.10 ${reflect * 0.4} 0" />
 	                <geometry>
 	                        <cylinder radius="0.2" length="0.05"/>
@@ -87,18 +91,12 @@
 	        </collision>
         </link>
-        <link name = "wheel_right">
-	        <visual>
-	                <!--<origin xyz="0 0 0" rpy="-0.0012068 0.114646 -0.0015308"/>-->
-	                <geometry>
-	                        <cylinder radius="0.2" length="0.05"/>
-	                </geometry>
- 	                </visual>
-	        <collision>
-	                <!--<origin xyz="0 0 0" rpy="-0.0012068 0.114646 -0.0015308"/> -->
-	                <geometry>
-	                        <cylinder radius="0.2" length="0.05"/>
-	                </geometry>
-	        </collision>
-        </link>
+        <joint name="wheel_${suffix}" type="continuous">
+                <origin xyz="-0.10 0.4 0.0" rpy="-1.57 0 0"/>
+                <parent link="base"/>
+                <child link="wheel_${suffix}"/>
+        </joint>
+</xacro:macro>
+<xacro:xacro_name suffix="left" reflect="1" />
+<xacro:xacro_name suffix="right" reflect="-1" />
         <link name = "wheel_center">
 	        <visual>
@@ -115,4 +113,10 @@
 	        </collision>
         </link>
+        <joint name="wheel_center" type="continuous">
+                <origin xyz="0.10 0 0" rpy="-1.57 0 0"/>
+                <parent link="base"/>
+                <child link="wheel_center"/>
+        </joint>
+ <!--JOINTS-->
          <joint name="base_laser_vert_bottom_joint" type="fixed">
                 <origin xyz="0.3158 -0.0021 0.5100" rpy="3.1355 -1.3045 0.0025"/>
@@ -135,18 +139,3 @@
                 <child link="laser_horiz"/>
         </joint>
-        <joint name="wheel_left" type="fixed">
-                <origin xyz="-0.10 0.4 0.0" rpy="-1.57 0 0"/>
-                <parent link="base"/>
-                <child link="wheel_left"/>
-        </joint>
-        <joint name="wheel_right" type="fixed">
-                <origin xyz="-0.10 -0.4 0" rpy="-1.57 0 0"/>
-                <parent link="base"/>
-                <child link="wheel_right"/>
-        </joint>
-        <joint name="wheel_center" type="fixed">
-                <origin xyz="0.10 0 0" rpy="-1.57 0 0"/>
-                <parent link="base"/>
-                <child link="wheel_center"/>
-        </joint>
 </robot>

Commit message: All three wheels on at the wrong orientation

File: urdf/robot.xacro (robot description, xacro)
@@ -91,8 +91,10 @@
 	        </collision>
         </link>
-        <joint name="wheel_${suffix}" type="continuous">
-                <origin xyz="-0.10 0.4 0.0" rpy="-1.57 0 0"/>
+        <joint name="wheel_${suffix}_joint" type="continuous">
+                <origin xyz="-0.10 0.4 0.0" rpy="0 0 -1.57"/>
                 <parent link="base"/>
                 <child link="wheel_${suffix}"/>
+                <!--<axis xyz = "0 0 1"/>-->
+                <!--weird things happening when axis added-->
         </joint>
 </xacro:macro>
@@ -113,8 +115,10 @@
 	        </collision>
         </link>
-        <joint name="wheel_center" type="continuous">
-                <origin xyz="0.10 0 0" rpy="-1.57 0 0"/>
+        <joint name="wheel_center_joint" type="continuous">
+                <origin xyz="0.10 0 0" rpy="0 0 -1.57"/>
                 <parent link="base"/>
                 <child link="wheel_center"/>
+                <axis xyz = "0 0 1"/>
+                <!--weird things happening when axis added-->
         </joint>
  <!--JOINTS-->

File: urdf/urdf_from_xacro.urdf (robot description, URDF)
Before this commit: robot robot, 8 links, 7 joints
Joints:
- removed joint wheel_center
- removed joint wheel_left
- removed joint wheel_right
- added joint wheel_center_joint: type continuous, parent base, child wheel_center, origin xyz=0.10 0 0 rpy=0 -1.57 0
- added joint wheel_left_joint: type continuous, parent base, child wheel_left, origin xyz=-0.10 0.4 0.0 rpy=0 0 -1.57
- added joint wheel_right_joint: type continuous, parent base, child wheel_right, origin xyz=-0.10 0.4 0.0 rpy=0 0 -1.57

Commit message: All three wheels on at the wrong orientation, robot disappeared when including other files section was included (first block of it. I cannot check if the second block is correct because the robot is gone)

File: urdf/robot.xacro (robot description, xacro)
@@ -1,4 +1,9 @@
 <?xml version="1.0"?>
 <robot xmlns:xacro="http://www.ros.org/wiki/xacro" name="robot">
+<!--INCLUDING OTHER FILES-->
+<!-- Include the XACRO file that defines a Hokuyo LIDAR. -->
+<xacro:include filename="$(find gazebo_plugins)/test/multi_robot_scenario/xacro/laser/hokuyo.xacro" />
+<!-- Include the XACRO file that defines a Hokuyo LIDAR. -->
+  <xacro:include filename="$(find velodyne_description)/urdf/VLP-16.urdf.xacro"/>
 <!--  position wrt parent == origin; orientation == rpy  -->
 <!--  units are in meters  -->
@@ -92,9 +97,8 @@
         </link>
         <joint name="wheel_${suffix}_joint" type="continuous">
-                <origin xyz="-0.10 0.4 0.0" rpy="0 0 -1.57"/>
+                <origin xyz="-0.10 ${reflect*0.4} 0.0" rpy="-1.57 0 0"/>
                 <parent link="base"/>
                 <child link="wheel_${suffix}"/>
-                <!--<axis xyz = "0 0 1"/>-->
-                <!--weird things happening when axis added-->
+                <axis xyz = "0 0 1"/>
         </joint>
 </xacro:macro>
@@ -116,16 +120,21 @@
         </link>
         <joint name="wheel_center_joint" type="continuous">
-                <origin xyz="0.10 0 0" rpy="0 0 -1.57"/>
+                <origin xyz="0.10 0 0" rpy="-1.57 0 0"/>
                 <parent link="base"/>
                 <child link="wheel_center"/>
                 <axis xyz = "0 0 1"/>
-                <!--weird things happening when axis added-->
         </joint>
  <!--JOINTS-->
-         <joint name="base_laser_vert_bottom_joint" type="fixed">
+ <!-- Include the XACRO file that defines a Hokuyo LIDAR. -->
+ <!--        <joint name="base_laser_vert_bottom_joint" type="fixed">
                 <origin xyz="0.3158 -0.0021 0.5100" rpy="3.1355 -1.3045 0.0025"/>
                 <parent link="base"/>
                 <child link="laser_vert_bottom"/>
         </joint>
+-->
+        <xacro:laser name="laser_vert_bottom" parent="base" xyz="0.3157894464801903
+        -0.002068548615034871 0.5099999434059285" rpy="3.1354753 -1.3045001 0.0024658"
+        meshes="package://gazebo_plugins/test/multi_robot_scenario/meshes/laser" />
+ <!--
         <joint name="base_laser_vert_top_right_joint" type="fixed">
                 <origin xyz="0.2978 -0.1450 1.8451" rpy="-1.1760 0.6313 1.9377"/>
@@ -133,4 +142,8 @@
                 <child link="laser_vert_top_right"/>
         </joint>
+-->
+        <xacro:laser name="laser_vert_top_right" parent="base" xyz="0.2978 -0.1450 1.8451" rpy="-1.1760 0.6313 1.9377"
+        meshes="package://gazebo_plugins/test/multi_robot_scenario/meshes/laser" />
+<!--
         <joint name="base_laser_vert_top_left_joint" type="fixed">
                 <origin xyz="0.2997 0.1531 1.8443" rpy="1.1780 0.6198 1.9560"/>
@@ -138,8 +151,18 @@
                 <child link="laser_vert_top_left"/>
         </joint>
-        <joint name="base_laser_horiz_joint" type="fixed">
+-->
+         <xacro:laser name="laser_vert_top_left" parent="base" xyz="0.2997 0.1531 1.8443" rpy="1.1780 0.6198     1.9560"
+        meshes="package://gazebo_plugins/test/multi_robot_scenario/meshes/laser" />
+<!--        <joint name="base_laser_horiz_joint" type="fixed">
                 <origin xyz="0.2325 0.0001 1.9201" rpy="-0.0012068 0.114646 -0.0015308"/>
                 <parent link="base"/>
                 <child link="laser_horiz"/>
         </joint>
+-->
+<!-- Invoke the macro to define the Hokuyo LIDAR. -->
+  <VLP-16 parent="base" name="laser_horiz" topic="laser_horiz/packets" hz="10"
+samples="440" gpu="false">
+       <origin xyz="0.2325416305773505 -0.0001380069427607134 1.920122926231907"
+rpy="-0.0012068 0.114646 -0.0015308" />
+  </VLP-16>
 </robot>

File: urdf/urdf_from_xacro.urdf (robot description, URDF)
Before this commit: robot robot, 8 links, 7 joints
Joints:
- joint wheel_center_joint: axis (none) -> 0 0 1; origin xyz=0.10 0 0 rpy=0 -1.57 0 -> xyz=0.10 0 0 rpy=-1.57 0 0
- joint wheel_left_joint: axis (none) -> 0 0 1; origin xyz=-0.10 0.4 0.0 rpy=0 0 -1.57 -> xyz=-0.10 0.4 0.0 rpy=-1.57 0 0
- joint wheel_right_joint: axis (none) -> 0 0 1; origin xyz=-0.10 0.4 0.0 rpy=0 0 -1.57 -> xyz=-0.10 -0.4 0.0 rpy=-1.57 0 0

Commit message: Final upload

File: urdf/robot.xacro (robot description, xacro)
@@ -24,7 +24,7 @@
 	        </collision>
         </link>
+<!--
         <link name = "laser_vert_bottom">
 	        <visual>
-	                <!--<origin xyz="0 0 0" rpy="3.1355 -1.3045 0.0025"/>-->
 	                <geometry>
 	                        <box size="0.062 0.062 0.087" />
@@ -32,5 +32,4 @@
  	        </visual>
 	        <collision>
-	                <!--<origin xyz="0 0 0" rpy="3.1355 -1.3045 0.0025"/>-->
 	                <geometry>
 	                        <box size="0.062 0.062 0.087" />
@@ -40,5 +39,4 @@
         <link name = "laser_vert_top_right">
 	        <visual>
-	                <!--<origin xyz="0 0 0" rpy="-1.1760 0.6313 1.9377"/>-->
 	                <geometry>
 	                        <box size="0.062 0.062 0.087" />
@@ -46,5 +44,4 @@
  	        </visual>
 	        <collision>
-	                <!--<origin xyz="0 0 0" rpy="-1.1760 0.6313 1.9377"/>-->
 	                <geometry>
 	                        <box size="0.062 0.062 0.087" />
@@ -54,5 +51,4 @@
         <link name = "laser_vert_top_left">
 	        <visual>
-	                <!--<origin xyz="0 0 0" rpy="1.1780 0.6198 1.9560"/>-->
 	                <geometry>
 	                        <box size="0.062 0.062 0.087" />
@@ -60,5 +56,4 @@
  	        </visual>
 	        <collision>
-	                <!--<origin xyz="0 0 0" rpy="1.1780 0.6198 1.9560"/>-->
 	                <geometry>
 	                        <box size="0.062 0.062 0.087" />
@@ -68,5 +63,4 @@
         <link name = "laser_horiz">
 	        <visual>
-	                <!--<origin xyz="0 0 0" rpy="-0.0012068 0.114646 -0.0015308"/>-->
 	                <geometry>
 	                        <cylinder radius="0.052" length="0.072"/>
@@ -74,5 +68,4 @@
  	                </visual>
 	        <collision>
-	                <!--<origin xyz="0 0 0" rpy="-0.0012068 0.114646 -0.0015308"/> -->
 	                <geometry>
 	                        <cylinder radius="0.052" length="0.072"/>
@@ -80,9 +73,9 @@
 	        </collision>
         </link>
+ -->
  <!--WHEELS-->
 <xacro:macro name="xacro_name" params="suffix reflect">
         <link name = "wheel_${suffix}">
 	        <visual>
-	                <origin xyz="-0.10 ${reflect * 0.4} 0" />
 	                <geometry>
 	                        <cylinder radius="0.2" length="0.05"/>
@@ -90,5 +83,4 @@
  	                </visual>
 	        <collision>
-	                <origin xyz="-0.10 ${reflect * 0.4} 0" />
 	                <geometry>
 	                        <cylinder radius="0.2" length="0.05"/>
@@ -97,5 +89,5 @@
         </link>
         <joint name="wheel_${suffix}_joint" type="continuous">
-                <origin xyz="-0.10 ${reflect*0.4} 0.0" rpy="-1.57 0 0"/>
+                <origin xyz="-0.10 ${reflect*0.4} 0.0" rpy="-${pi/2} 0 0"/>
                 <parent link="base"/>
                 <child link="wheel_${suffix}"/>
@@ -120,5 +112,5 @@
         </link>
         <joint name="wheel_center_joint" type="continuous">
-                <origin xyz="0.10 0 0" rpy="-1.57 0 0"/>
+                <origin xyz="0.10 0 0" rpy="-${pi/2} 0 0"/>
                 <parent link="base"/>
                 <child link="wheel_center"/>

File: urdf/urdf_from_xacro.urdf (robot description, URDF)
Before this commit: robot robot, 8 links, 7 joints
Links:
- added link laser_horiz_base_link, mass 0.83; collision cylinder length=0.0717 radius=0.0516; visual mesh filename=package://velodyne_description/meshes/VLP16_base_1.dae
- link laser_horiz: mass None -> 0.01; geometry visual mesh filename=package://velodyne_description/meshes/VLP16_scan.dae
- link laser_vert_bottom: mass None -> 1e-5; geometry collision box size=0.1 0.1 0.1; visual mesh filename=package://gazebo_plugins/test/multi_robot_scenario/meshes/l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
- link laser_vert_top_left: mass None -> 1e-5; geometry collision box size=0.1 0.1 0.1; visual mesh filename=package://gazebo_plugins/test/multi_robot_scenario/meshes/l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
- link laser_vert_top_right: mass None -> 1e-5; geometry collision box size=0.1 0.1 0.1; visual mesh filename=package://gazebo_plugins/test/multi_robot_scenario/meshes/l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
Joints:
- removed joint base_laser_horiz_joint
- added joint laser_horiz_base_mount_joint: type fixed, parent base, child laser_horiz_base_link, origin xyz=0.2325416305773505 -0.0001380069427607134 1.920122926231907 rpy=-0.0012068 0.114646 -0.0015308
- added joint laser_horiz_base_scan_joint: type fixed, parent laser_horiz_base_link, child laser_horiz, origin xyz=0 0 0.0377 rpy=0 0 0
- joint base_laser_vert_bottom_joint: axis (none) -> 0 0 1; origin xyz=0.3158 -0.0021 0.5100 rpy=3.1355 -1.3045 0.0025 -> xyz=0.3157894464801903         -0.002068548615034871 0.5099999434059285 rpy=3.1354753 -1.3045001 0.0024658
- joint base_laser_vert_top_left_joint: axis (none) -> 0 0 1; origin xyz=0.2997 0.1531 1.8443 rpy=1.1780 0.6198 1.9560 -> xyz=0.2997 0.1531 1.8443 rpy=1.1780 0.6198     1.9560
- joint base_laser_vert_top_right_joint: axis (none) -> 0 0 1
- joint wheel_center_joint: origin xyz=0.10 0 0 rpy=-1.57 0 0 -> xyz=0.10 0 0 rpy=-1.57079632679 0 0
- joint wheel_left_joint: origin xyz=-0.10 0.4 0.0 rpy=-1.57 0 0 -> xyz=-0.10 0.4 0.0 rpy=-1.57079632679 0 0
- joint wheel_right_joint: origin xyz=-0.10 -0.4 0.0 rpy=-1.57 0 0 -> xyz=-0.10 -0.4 0.0 rpy=-1.57079632679 0 0
